File: hardware/ro-antena-array/_autosave-ro-antena-array.kicad_pcb (KiCad board)
At the start: 2 copper layers, 83 x 350.9 mm, 15 parts

Commit message: main: hardware: ro-antenna-array project beginnig
Changed lines of the file:
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@@
 	(gr_poly
 		(pts
-			(xy 217.2 193.4) (xy 224.2 186.4) (xy 260.2 186.4) (xy 267.2 193.4) (xy 267.2 230.4) (xy 260.2 236.4)
-			(xy 223.2 236.4) (xy 217.2 229.4)
+			(xy 217.2 103.753) (xy 229.7 91.253) (xy 254.7 91.253) (xy 267.2 103.753) (xy 267.2 128.753) (xy 254.7 141.253)
+			(xy 229.7 141.253) (xy 217.2 128.753)
 		)
 		(stroke
@@
 	(gr_poly
 		(pts
-			(xy 217.2 288.547) (xy 224.2 281.547) (xy 260.2 281.547) (xy 267.2 288.547) (xy 267.2 325.547) (xy 260.2 331.547)
-			(xy 223.2 331.547) (xy 217.2 324.547)
+			(xy 217.2 294.047) (xy 229.7 281.547) (xy 254.7 281.547) (xy 267.2 294.047) (xy 267.2 319.047) (xy 254.7 331.547)
+			(xy 229.7 331.547) (xy 217.2 319.047)
 		)
 		(stroke
@@
 	(gr_poly
 		(pts
-			(xy 217.2 98.253) (xy 224.2 91.253) (xy 260.2 91.253) (xy 267.2 98.253) (xy 267.2 135.253) (xy 260.2 141.253)
-			(xy 223.2 141.253) (xy 217.2 134.253)
+			(xy 217.2 198.9) (xy 229.7 186.4) (xy 254.7 186.4) (xy 267.2 198.9) (xy 267.2 223.9) (xy 254.7 236.4)
+			(xy 229.7 236.4) (xy 217.2 223.9)
 		)
 		(stroke
@@
 	(gr_poly
 		(pts
-			(xy 217.2 98.253) (xy 224.2 91.253) (xy 260.2 91.253) (xy 267.2 98.253) (xy 267.2 135.253) (xy 260.2 141.253)
-			(xy 223.2 141.253) (xy 217.2 134.253)
+			(xy 217.2 294.047) (xy 229.7 281.547) (xy 254.7 281.547) (xy 267.2 294.047) (xy 267.2 319.047) (xy 254.7 331.547)
+			(xy 229.7 331.547) (xy 217.2 319.047)
 		)
 		(stroke
@@
 	(gr_poly
 		(pts
-			(xy 217.2 193.4) (xy 224.2 186.4) (xy 260.2 186.4) (xy 267.2 193.4) (xy 267.2 230.4) (xy 260.2 236.4)
-			(xy 223.2 236.4) (xy 217.2 229.4)
+			(xy 217.2 103.753) (xy 229.7 91.253) (xy 254.7 91.253) (xy 267.2 103.753) (xy 267.2 128.753) (xy 254.7 141.253)
+			(xy 229.7 141.253) (xy 217.2 128.753)
 		)
 		(stroke
@@
 	(gr_poly
 		(pts
-			(xy 217.2 288.547) (xy 224.2 281.547) (xy 260.2 281.547) (xy 267.2 288.547) (xy 267.2 325.547) (xy 260.2 331.547)
-			(xy 223.2 331.547) (xy 217.2 324.547)
+			(xy 217.2 198.9) (xy 229.7 186.4) (xy 254.7 186.4) (xy 267.2 198.9) (xy 267.2 223.9) (xy 254.7 236.4)
+			(xy 229.7 236.4) (xy 217.2 223.9)
 		)
 		(stroke
